File: _autosave-lipo_Charger.kicad_pcb (KiCad board)
At the start: 2 copper layers, 45 parts, among them Q1 NVTFS010N10MCLTAG(high power), Q2 NVTFS010N10MCLTAG(high power), Q3 NVTFS010N10MCLTAG(high power), Q4 NVTFS010N10MCLTAG(high power), U1 BQ25703ARSNR

Commit message: three r one c balancing circuit dev board has to be done yet
Parts:
- added L1: 2.2uh, Inductor_SMD:L_10.4x10.4_H4.8, F.Cu at (121.6, 66.6)
- moved U1 2.77 mm to (132.7, 104.9)
Connections:
- Q1 pad 1-2-3: Net-(MOSFET1-D-Pad5) -> Net-(U1-SW2)
- Q1 pad 5-6-7-8: Net-(U1-SW2) -> Net-(MOSFET1-D-Pad5)
- Q4 pad 1-2-3: Net-(U1-SW2) -> GND
- Q4 pad 5-6-7-8: GND -> Net-(U1-SW2)
