File: lipo_Charger.kicad_sch (KiCad schematic)
At the start: 111 parts, among them J1 XT60PW-M, J2 Conn_01x01, J3 balance_plug_4s, J4 Conn_01x05, J5 Conn_01x04, J6 Conn_01x01, J7 Conn_01x07, J8 Conn_01x04, Q1 NX7002AK_215(nch low power), Q2 NVTFS010N10MCLTAG(high power)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

Commit message: sch organized a bit
Other:
- note added: "balancing circuit"
- note added: "cell voltage level monitor (adc)"
- note added: "charging circuit"
- note added: "led_ indications"
- moved on the sheet: C30, C31, C32, C33, C34, D1, D2, D3, D4, J4, J5, J8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

Commit message: final correction has been ready to order
Parts:
- removed D3, D4: LED, LED_THT:LED_D5.0mm, symbol Device:LED
- removed J8: Conn_01x04, Connector_PinHeader_2.54mm:PinHeader_1x04_P2.54mm_Vertical, symbol Connector_Generic:Conn_01x04
- removed R38, R42: R, Resistor_THT:R_Axial_DIN0204_L3.6mm_D1.6mm_P5.08mm_Horizontal, symbol Device:R
- added J10, J11, J12, J9: Conn_01x20, Connector_PinHeader_2.54mm:PinHeader_1x20_P2.54mm_Vertical, symbol Connector_Generic:Conn_01x20
- added J13: Conn_01x02, Connector_PinHeader_2.54mm:PinHeader_1x02_P2.54mm_Vertical, symbol Connector_Generic:Conn_01x02
Connections:
- net BAT_adc: now also J12.11 (Pin_11), J9.11 (Pin_11)
- net CELL_1S_adc: now also J12.15 (Pin_15), J9.15 (Pin_15)
- net CELL_2S_adc: now also J12.14 (Pin_14), J9.14 (Pin_14)
- net CELL_3S_adc: now also J12.13 (Pin_13), J9.13 (Pin_13)
- net CELL_4S_adc: now also J12.12 (Pin_12), J9.12 (Pin_12)
- net CHRG_OK: now also J12.8 (Pin_8), J9.8 (Pin_8)
- net CMPOUT: now also J12.6 (Pin_6), J9.6 (Pin_6)
- net EN_OTG: now also J12.9 (Pin_9), J9.9 (Pin_9)
- net GNDA: now also J10.19 (Pin_19), J11.19 (Pin_19), J12.2 (Pin_2), J9.2 (Pin_2)
- net ILIM_HIZ: now also J12.10 (Pin_10), J9.10 (Pin_10)
- net VDDA: now also J10.20 (Pin_20), J11.20 (Pin_20), J12.3 (Pin_3), J9.3 (Pin_3)
- net 2SGATE: now reaches J5.2 (Pin_2), Q7.1, R15.1
- net 2SGATE: now also J10.16 (Pin_16), J11.16 (Pin_16)
- net 1SGATE: now reaches J5.1 (Pin_1), Q8.1, R21.1
- net 1SGATE: now also J10.17 (Pin_17), J11.17 (Pin_17)
- net at R22.1: now also J13.2 (Pin_2)
- net 3SGATE: now reaches J5.3 (Pin_3), Q6.1, R9.1
- net 3SGATE: now also J10.15 (Pin_15), J11.15 (Pin_15)
- net 4SGATE: now reaches J5.4 (Pin_4), Q1.1, R3.1
- net 4SGATE: now also J10.14 (Pin_14), J11.14 (Pin_14)
- net at R14.1: now also J13.1 (Pin_1)
- net PROCHOT_N renamed PB0
- net PB0: now also J12.7 (Pin_7), J9.7 (Pin_7)
- net SCL renamed PB10
- net PB10: now also J12.4 (Pin_4), J9.4 (Pin_4)
- net SDA renamed PB3
- net PB3: now also J10.11 (Pin_11), J11.11 (Pin_11)
- new net 5V: J10.18 (Pin_18), J11.18 (Pin_18), J12.1 (Pin_1), J9.1 (Pin_1)
- new net PA10: J10.7 (Pin_7), J11.7 (Pin_7)
- new net PA11: J10.8 (Pin_8), J11.8 (Pin_8)
- new net PA12: J10.9 (Pin_9), J11.9 (Pin_9)
- new net PA15: J10.10 (Pin_10), J11.10 (Pin_10)
- new net PA8: J10.5 (Pin_5), J11.5 (Pin_5)
- new net PA9: J10.6 (Pin_6), J11.6 (Pin_6)
- new net PB12: J10.1 (Pin_1), J11.1 (Pin_1)
- new net PB13: J10.2 (Pin_2), J11.2 (Pin_2)
- new net PB14: J10.3 (Pin_3), J11.3 (Pin_3)
- new net PB15: J10.4 (Pin_4), J11.4 (Pin_4)
- new net PB2: J12.5 (Pin_5), J9.5 (Pin_5)
- new net PB4: J10.12 (Pin_12), J11.12 (Pin_12)
- new net PB5: J10.13 (Pin_13), J11.13 (Pin_13)
- new net PC13: J12.19 (Pin_19), J9.19 (Pin_19)
- new net PC14: J12.18 (Pin_18), J9.18 (Pin_18)
- new net PC15: J12.17 (Pin_17), J9.17 (Pin_17)
- new net RESET: J12.16 (Pin_16), J9.16 (Pin_16)
- new net VBAT: J12.20 (Pin_20), J9.20 (Pin_20)

Commit message: final ordered file
Connections:
- net 1SGATE: now also J10.14 (Pin_14), J11.14 (Pin_14); no longer J10.17 (Pin_17), J11.17 (Pin_17)
- net 2SGATE: now also J10.15 (Pin_15), J11.15 (Pin_15); no longer J10.16 (Pin_16), J11.16 (Pin_16)
- net 3SGATE: now also J10.16 (Pin_16), J11.16 (Pin_16); no longer J10.15 (Pin_15), J11.15 (Pin_15)
- net 4SGATE: now also J10.17 (Pin_17), J11.17 (Pin_17); no longer J10.14 (Pin_14), J11.14 (Pin_14)
Changed lines of the file:
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@@
 		)
 	)
-	(text_box "stm32 dev board\n"
-		(exclude_from_sim no)
-		(at 72.39 449.58 0)
-		(size 207.01 116.84)
-		(margins 0.9525 0.9525 0.9525 0.9525)
-		(stroke
-			(width 0)
-			(type solid)
-		)
-		(fill
-			(type none)
-		)
-		(effects
-			(font
-				(size 1.27 1.27)
-			)
-			(justify left top)
-		)
-	)
 	(junction
 		(at 120.65 109.22)
@@
 	)
 	(label "4SGATE"
-		(at 130.81 515.62 0)
+		(at 130.81 523.24 0)
 		(effects
 			(font
@@
 	)
 	(label "3SGATE"
-		(at 130.81 518.16 0)
+		(at 130.81 520.7 0)
 		(effects
 			(font
@@
 	)
 	(label "2SGATE"
-		(at 130.81 520.7 0)
+		(at 130.81 518.16 0)
 		(effects
 			(font
@@
 	)
 	(label "1SGATE"
-		(at 130.81 523.24 0)
+		(at 130.81 515.62 0)
 		(effects
 			(font
